File: PCB/Main_Board/Main_Board.sch (KiCad schematic (older format))
At the start: 14 parts, among them J1 USB_B_Micro, J2 Screw_Terminal_01x02, J3 Screw_Terminal_01x01, J4 AudioJack3, J5 AudioJack3, SW1 SW_SPDT, U1 TLV75533PDBV

Commit message: Add IR circuit
Parts:
- added U2: TSSP58P38, OptoDevice:Vishay_MINICAST-3Pin, symbol Sensor_Proximity:TSSP58P38
- renumbered J4 to J3, J5 to J4, J3 to J5
Connections:
- net labels added: IR_SENSOR
- wire segments 108 -> 111
- no-connect marks 19 -> 18

Commit message: Further schematic work and footprint association
Parts:
- removed J3, J4: AudioJack3, symbol Connector:AudioJack3
- removed J5: Screw_Terminal_01x01, symbol Connector:Screw_Terminal_01x01
- removed U2: TSSP58P38, OptoDevice:Vishay_MINICAST-3Pin, symbol Sensor_Proximity:TSSP58P38
- added J3, J4: SJ1-3523N, SamacSys:SJ13523N, symbol SamacSys:SJ1-3523N
- added J5: Screw_Terminal_01x04, symbol Connector:Screw_Terminal_01x04
- C1, C2: footprint (none) -> Capacitor_SMD:C_0603_1608Metric_Pad1.05x0.95mm_HandSolder
- D4: footprint (none) -> LED_SMD:LED_0603_1608Metric_Pad1.05x0.95mm_HandSolder
- J1: footprint (none) -> Connector_USB:USB_Micro-B_Amphenol_10103594-0001LF_Horizontal; Product (none) -> https://www.mouser.co.uk/ProductDetail/Amphenol-FCI/1011819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
- R1: footprint (none) -> Resistor_SMD:R_0603_1608Metric_Pad1.05x0.95mm_HandSolder
- SW1: footprint (none) -> SamacSys:CS12ANW03; Product (none) -> https://www.mouser.co.uk/ProductDetail/NKK-Switches/CS12ANW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
Connections:
- no-connect marks 18 -> 22
Changed lines of the file:
@@
 F 0 "J1" H 1207 2567 50  0000 C CNN
 F 1 "USB_B_Micro" H 1207 2476 50  0000 C CNN
-F 2 "" H 1300 2050 50  0001 C CNN
+F 2 "Connector_USB:USB_Micro-B_Amphenol_10103594-0001LF_Horizontal" H 1300 2050 50  0001 C CNN
 F 3 "~" H 1300 2050 50  0001 C CNN
+F 4 "https://www.mouser.co.uk/ProductDetail/Amphenol-FCI/10118194-0001LF?qs=Ywefl8B65e4FIdY8OWfRQA%3D%3D" H 1150 2100 50  0001 C CNN "Product"
 	1    1150 2100
 	1    0    0    -1
@@
 F 0 "D4" H 2450 4485 50  0000 C CNN
 F 1 "3V3_LED" H 2450 4394 50  0000 C CNN
-F 2 "" V 2450 4250 50  0001 C CNN
+F 2 "LED_SMD:LED_0603_1608Metric_Pad1.05x0.95mm_HandSolder" V 2450 4250 50  0001 C CNN
 F 3 "~" V 2450 4250 50  0001 C CNN
 	1    2450 4250
@@
 F 0 "R1" H 2509 4546 50  0000 L CNN
 F 1 "CUR_LIMIT" H 2509 4455 50  0000 L CNN
-F 2 "" H 2450 4500 50  0001 C CNN
+F 2 "Resistor_SMD:R_0603_1608Metric_Pad1.05x0.95mm_HandSolder" H 2450 4500 50  0001 C CNN
 F 3 "~" H 2450 4500 50  0001 C CNN
 	1    2450 4500
@@
 F 0 "SW1" V 1246 3462 50  0000 R CNN
 F 1 "SW_SPDT" V 1155 3462 50  0000 R CNN
-F 2 "" H 1200 3650 50  0001 C CNN
+F 2 "SamacSys:CS12ANW03" H 1200 3650 50  0001 C CNN
 F 3 "~" H 1200 3650 50  0001 C CNN
+F 4 "https://www.mouser.co.uk/ProductDetail/NKK-Switches/CS12ANW03?qs=4P1McwaGddbVHu%252BBZT0egw%3D%3D" V 1200 3650 50  0001 C CNN "Product"
 	1    1200 3650
 	0    -1   -1   0
@@
 F 0 "C1" H 1442 4546 50  0000 L CNN
 F 1 "10uF" H 1442 4455 50  0000 L CNN
-F 2 "" H 1350 4500 50  0001 C CNN
+F 2 "Capacitor_SMD:C_0603_1608Metric_Pad1.05x0.95mm_HandSolder" H 1350 4500 50  0001 C CNN
 F 3 "~" H 1350 4500 50  0001 C CNN
 	1    1350 4500
@@
 F 0 "C2" H 2242 4546 50  0000 L CNN
 F 1 "10uF" H 2242 4455 50  0000 L CNN
-F 2 "" H 2150 4500 50  0001 C CNN
+F 2 "Capacitor_SMD:C_0603_1608Metric_Pad1.05x0.95mm_HandSolder" H 2150 4500 50  0001 C CNN
 F 3 "~" H 2150 4500 50  0001 C CNN
 	1    2150 4500
@@
 Text Label 6100 2400 2    50   ~ 0
 MSGEQ7_STROBE
-$Comp
-L Connector:Screw_Terminal_01x01 J5
-U 1 1 5FB21930
-P 6450 3250
-F 0 "J5" H 6530 3292 50  0000 L CNN
-F 1 "Screw_Terminal_01x01" H 6530 3201 50  0000 L CNN
-F 2 "" H 6450 3250 50  0001 C CNN
-F 3 "~" H 6450 3250 50  0001 C CNN
-	1    6450 3250
-	1    0    0    -1
-$EndComp
-Text Label 6150 3250 2    50   ~ 0
+Text Label 4250 4650 0    50   ~ 0
 LED_OUT
-Wire Wire Line
-	6150 3250 6250 3250
 Text Label 4700 3050 0    50   ~ 0
 MSGEQ7_L_OUT
@@
 	4500 1550 4700 1550
 $Comp
-L Connector:AudioJack3 J3
-U 1 1 5FB5ADE2
-P 6100 3800
-F 0 "J3" H 6082 4125 50  0000 C CNN
-F 1 "AudioJack3" H 6082 4034 50  0000 C CNN
-F 2 "" H 6100 3800 50  0001 C CNN
-F 3 "~" H 6100 3800 50  0001 C CNN
-	1    6100 3800
-	1    0    0    -1
-$EndComp
-$Comp
-L power:Earth #PWR07
-U 1 1 5FB5D663
-P 6400 4600
-AR Path="/5FB5D663" Ref="#PWR07"  Part="1"
-AR Path="/5F591C5D/5FB5D663" Ref="#PWR?"  Part="1"
-F 0 "#PWR07" H 6400 4350 50  0001 C CNN
-F 1 "Earth" H 6400 4450 50  0001 C CNN
-F 2 "" H 6400 4600 50  0001 C CNN
-F 3 "~" H 6400 4600 50  0001 C CNN
-	1    6400 4600
-	1    0    0    -1
-$EndComp
-Text Label 6600 3900 0    50   ~ 0
-AUDIO_L
-Text Label 6600 3800 0    50   ~ 0
-AUDIO_R
-Wire Wire Line
-	6400 3700 6300 3700
-$Comp
-L Connector:AudioJack3 J4
-U 1 1 5FB76A93
-P 6100 4400
-F 0 "J4" H 6082 4725 50  0000 C CNN
-F 1 "AudioJack3" H 6082 4634 50  0000 C CNN
-F 2 "" H 6100 4400 50  0001 C CNN
-F 3 "~" H 6100 4400 50  0001 C CNN
-	1    6100 4400
-	1    0    0    -1
-$EndComp
-Wire Wire Line
-	6400 3700 6400 4300
-Wire Wire Line
-	6300 4300 6400 4300
-Connection ~ 6400 4300
-Wire Wire Line
-	6400 4300 6400 4600
-Wire Wire Line
-	6300 3800 6450 3800
-Wire Wire Line
-	6450 3800 6450 4400
-Wire Wire Line
-	6450 4400 6300 4400
-Wire Wire Line
-	6300 3900 6500 3900
-Wire Wire Line
-	6500 3900 6500 4500
-Wire Wire Line
-	6500 4500 6300 4500
-Wire Wire Line
-	6600 3800 6450 3800
-Connection ~ 6450 3800
-Wire Wire Line
-	6500 3900 6600 3900
-Connection ~ 6500 3900
-$Comp
-L Sensor_Proximity:TSSP58P38 U2
-U 1 1 5F555A66
-P 4350 4350
-F 0 "U2" H 4338 4775 50  0000 C CNN
-F 1 "TSSP58P38" H 4338 4684 50  0000 C CNN
-F 2 "OptoDevice:Vishay_MINICAST-3Pin" H 4300 3975 50  0001 C CNN
-F 3 "http://www.vishay.com/docs/82462/tsop581.pdf" H 5000 4650 50  0001 C CNN
-	1    4350 4350
-	1    0    0    -1
-$EndComp
-$Comp
 L power:Earth #PWR05
 U 1 1 5F55AF8B
-P 4850 4550
+P 4650 4350
 AR Path="/5F55AF8B" Ref="#PWR05"  Part="1"
 AR Path="/5F591C5D/5F55AF8B" Ref="#PWR?"  Part="1"
-F 0 "#PWR05" H 4850 4300 50  0001 C CNN
-F 1 "Earth" H 4850 4400 50  0001 C CNN
-F 2 "" H 4850 4550 50  0001 C CNN
-F 3 "~" H 4850 4550 50  0001 C CNN
-	1    4850 4550
+F 0 "#PWR05" H 4650 4100 50  0001 C CNN
+F 1 "Earth" H 4650 4200 50  0001 C CNN
+F 2 "" H 4650 4350 50  0001 C CNN
+F 3 "~" H 4650 4350 50  0001 C CNN
+	1    4650 4350
 	0    -1   -1   0
 $EndComp
-Text Label 4850 4150 0    50   ~ 0
+Text Label 4250 4550 0    50   ~ 0
 +3.3V
-Wire Wire Line
-	4850 4150 4750 4150
-Wire Wire Line
-	4750 4550 4850 4550
 Text Label 4700 2950 0    50   ~ 0
 IR_SENSOR
 Wire Wire Line
 	4500 2950 4700 2950
-Text Label 4850 4350 0    50   ~ 0
+Text Label 4250 4450 0    50   ~ 0
 IR_SENSOR
-Wire Wire Line
-	4850 4350 4750 4350
+$Comp
+L SamacSys:SJ1-3523N J3
+U 1 1 5F5CB765
+P 5400 4000
+F 0 "J3" H 6100 4265 50  0000 C CNN
+F 1 "SJ1-3523N" H 6100 4174 50  0000 C CNN
+F 2 "SamacSys:SJ13523N" H 6650 4100 50  0001 L CNN
+F 3 "https://componentsearchengine.com/Datasheets/1/SJ1-3523N.pdf" H 6650 4000 50  0001 L CNN
+F 4 "Phone Connectors 3.5 MM AUDIO JACK" H 6650 3900 50  0001 L CNN "Description"
+F 5 "5.5" H 6650 3800 50  0001 L CNN "Height"
+F 6 "490-SJ1-3523N" H 6650 3700 50  0001 L CNN "Mouser Part Number"
+F 7 "https://www.mouser.co.uk/ProductDetail/CUI-Devices/SJ1-3523N?qs=WyjlAZoYn50aNl0vAhb3Tg%3D%3D" H 6650 3600 50  0001 L CNN "Mouser Price/Stock"
+F 8 "CUI Devices" H 6650 3500 50  0001 L CNN "Manufacturer_Name"
+F 9 "SJ1-3523N" H 6650 3400 50  0001 L CNN "Manufacturer_Part_Number"
+	1    5400 4000
+	1    0    0    -1
+$EndComp
+$Comp
+L SamacSys:SJ1-3523N J4
+U 1 1 5F5DC996
+P 5400 4800
+F 0 "J4" H 6100 5065 50  0000 C CNN
+F 1 "SJ1-3523N" H 6100 4974 50  0000 C CNN
+F 2 "SamacSys:SJ13523N" H 6650 4900 50  0001 L CNN
+F 3 "https://componentsearchengine.com/Datasheets/1/SJ1-3523N.pdf" H 6650 4800 50  0001 L CNN
+F 4 "Phone Connectors 3.5 MM AUDIO JACK" H 6650 4700 50  0001 L CNN "Description"
+F 5 "5.5" H 6650 4600 50  0001 L CNN "Height"
+F 6 "490-SJ1-3523N" H 6650 4500 50  0001 L CNN "Mouser Part Number"
+F 7 "https://www.mouser.co.uk/ProductDetail/CUI-Devices/SJ1-3523N?qs=WyjlAZoYn50aNl0vAhb3Tg%3D%3D" H 6650 4400 50  0001 L CNN "Mouser Price/Stock"
+F 8 "CUI Devices" H 6650 4300 50  0001 L CNN "Manufacturer_Name"
+F 9 "SJ1-3523N" H 6650 4200 50  0001 L CNN "Manufacturer_Part_Number"
+	1    5400 4800
+	1    0    0    -1
+$EndComp
+$Comp
+L power:Earth #PWR07
+U 1 1 5F5E0067
+P 5700 4900
+AR Path="/5F5E0067" Ref="#PWR07"  Part="1"
+AR Path="/5F591C5D/5F5E0067" Ref="#PWR?"  Part="1"
+F 0 "#PWR07" H 5700 4650 50  0001 C CNN
+F 1 "Earth" H 5700 4750 50  0001 C CNN
+F 2 "" H 5700 4900 50  0001 C CNN
+F 3 "~" H 5700 4900 50  0001 C CNN
+	1    5700 4900
+	1    0    0    -1
+$EndComp
+Wire Wire Line
+	5800 4000 5700 4000
+Wire Wire Line
+	5700 4000 5700 4800
+Connection ~ 5700 4800
+Wire Wire Line
+	5700 4800 5700 4900
+Wire Wire Line
+	5700 4800 5800 4800
+Text Label 7050 4000 0    50   ~ 0
+AUDIO_R
+Wire Wire Line
+	6800 4000 6900 4000
+Wire Wire Line
+	6800 4800 6900 4800
+Wire Wire Line
+	6900 4800 6900 4000
+Connection ~ 6900 4000
+Text Label 7050 4300 0    50   ~ 0
+AUDIO_L
+Wire Wire Line
+	6800 5100 6950 5100
+Wire Wire Line
+	6950 5100 6950 4300
+Wire Wire Line
+	6950 4300 7050 4300
+Wire Wire Line
+	6800 4300 6950 4300
+Connection ~ 6950 4300
+Wire Wire Line
+	6900 4000 7050 4000
+NoConn ~ 6800 4100
+NoConn ~ 6800 4200
+NoConn ~ 6800 4900
+NoConn ~ 6800 5000
+$Comp
+L Connector:Screw_Terminal_01x04 J5
+U 1 1 5F654BAB
+P 3950 4550
+F 0 "J5" H 3868 4125 50  0000 C CNN
+F 1 "Screw_Terminal_01x04" H 3868 4216 50  0000 C CNN
+F 2 "" H 3950 4550 50  0001 C CNN
+F 3 "~" H 3950 4550 50  0001 C CNN
+	1    3950 4550
+	-1   0    0    1
+$EndComp
+Wire Wire Line
+	4150 4350 4650 4350
+Wire Wire Line
+	4150 4450 4250 4450
+Wire Wire Line
+	4150 4550 4250 4550
+Wire Wire Line
+	4150 4650 4250 4650
 $EndSCHEMATC

Commit message: Further sourcing on mouser
Parts:
- removed D1, D2, D3: D_TVS, symbol Device:D_TVS
- J2: footprint (none) -> TerminalBlock:TerminalBlock_bornier-2_P5.08mm; Product (none) -> https://www.mouser.co.uk/ProductDetail/CUI-Devices/TB006-50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
- J5: footprint (none) -> TerminalBlock:TerminalBlock_bornier-4_P5.08mm; Product (none) -> https://www.mouser.co.uk/ProductDetail/CUI-Devices/TB006-50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
- R1: value CUR_LIMIT -> CUR_LIMIT_5.6R
Connections:
- wire segments 111 -> 98
Changed lines of the file:
@@
 NoConn ~ 1450 2300
 Connection ~ 1150 2550
-Wire Wire Line
-	2400 1900 2450 1900
-$Comp
-L Device:D_TVS D1
-U 1 1 5F884D02
-P 1600 2400
-AR Path="/5F884D02" Ref="D1"  Part="1"
-AR Path="/5F591C5D/5F884D02" Ref="D?"  Part="1"
-F 0 "D1" V 1554 2479 50  0000 L CNN
-F 1 "D_TVS" V 1645 2479 50  0000 L CNN
-F 2 "" H 1600 2400 50  0001 C CNN
-F 3 "~" H 1600 2400 50  0001 C CNN
-	1    1600 2400
-	0    1    1    0
-$EndComp
-$Comp
-L Device:D_TVS D2
-U 1 1 5F884D08
-P 2000 2400
-AR Path="/5F884D08" Ref="D2"  Part="1"
-AR Path="/5F591C5D/5F884D08" Ref="D?"  Part="1"
-F 0 "D2" V 1954 2479 50  0000 L CNN
-F 1 "D_TVS" V 2045 2479 50  0000 L CNN
-F 2 "" H 2000 2400 50  0001 C CNN
-F 3 "~" H 2000 2400 50  0001 C CNN
-	1    2000 2400
-	0    1    1    0
-$EndComp
-$Comp
-L Device:D_TVS D3
-U 1 1 5F884D0E
-P 2400 2400
-AR Path="/5F884D0E" Ref="D3"  Part="1"
-AR Path="/5F591C5D/5F884D0E" Ref="D?"  Part="1"
-F 0 "D3" V 2354 2479 50  0000 L CNN
-F 1 "D_TVS" V 2445 2479 50  0000 L CNN
-F 2 "" H 2400 2400 50  0001 C CNN
-F 3 "~" H 2400 2400 50  0001 C CNN
-	1    2400 2400
-	0    1    1    0
-$EndComp
-Wire Wire Line
-	1600 2550 1600 2600
-Wire Wire Line
-	1600 2600 2000 2600
-Wire Wire Line
-	2400 2600 2400 2550
-Wire Wire Line
-	2000 2550 2000 2600
-Connection ~ 2000 2600
-Wire Wire Line
-	2000 2600 2400 2600
-Wire Wire Line
-	2400 1900 2400 2250
-Wire Wire Line
-	2000 2250 2000 2100
-Wire Wire Line
-	2000 2100 1450 2100
-Wire Wire Line
-	1450 2200 1600 2200
-Wire Wire Line
-	1600 2200 1600 2250
-Wire Wire Line
-	1150 2550 1150 2600
-Wire Wire Line
-	1600 2600 1150 2600
-Connection ~ 1600 2600
-Connection ~ 1150 2600
-Connection ~ 2400 1900
-Wire Wire Line
-	2000 2100 2450 2100
-Connection ~ 2000 2100
-Wire Wire Line
-	1600 2200 2450 2200
-Connection ~ 1600 2200
-Text Label 2450 2100 0    50   ~ 0
+Text Label 1750 2100 0    50   ~ 0
 D+
-Text Label 2450 2200 0    50   ~ 0
+Text Label 1750 2200 0    50   ~ 0
 D-
-Wire Wire Line
-	1150 2600 1150 2700
 Wire Wire Line
 	1750 4650 2150 4650
@@
 AR Path="/5F591C5D/5F884D5C" Ref="R?"  Part="1"
 F 0 "R1" H 2509 4546 50  0000 L CNN
-F 1 "CUR_LIMIT" H 2509 4455 50  0000 L CNN
+F 1 "CUR_LIMIT_5.6R" H 2509 4455 50  0000 L CNN
 F 2 "Resistor_SMD:R_0603_1608Metric_Pad1.05x0.95mm_HandSolder" H 2450 4500 50  0001 C CNN
 F 3 "~" H 2450 4500 50  0001 C CNN
@@
 Wire Wire Line
 	1300 3400 1300 3450
-Text Label 2450 1900 0    50   ~ 0
+Text Label 1750 1900 0    50   ~ 0
 +USB_5V
 Text Label 1300 3400 1    50   ~ 0
@@
 F 0 "J2" H 1168 1517 50  0000 C CNN
 F 1 "Screw_Terminal_01x02" H 1168 1426 50  0000 C CNN
-F 2 "" H 1250 1300 50  0001 C CNN
+F 2 "TerminalBlock:TerminalBlock_bornier-2_P5.08mm" H 1250 1300 50  0001 C CNN
 F 3 "~" H 1250 1300 50  0001 C CNN
+F 4 "https://www.mouser.co.uk/ProductDetail/CUI-Devices/TB006-508-02BE?qs=vLWxofP3U2wEdOVV%2FaT04w%3D%3D" H 1250 1300 50  0001 C CNN "Product"
 	1    1250 1300
 	-1   0    0    -1
@@
 	1550 1300 1500 1300
 Connection ~ 1500 1300
-Wire Wire Line
-	1450 1900 2400 1900
 $Comp
 L power:PWR_FLAG #FLG01
@@
 F 0 "J5" H 3868 4125 50  0000 C CNN
 F 1 "Screw_Terminal_01x04" H 3868 4216 50  0000 C CNN
-F 2 "" H 3950 4550 50  0001 C CNN
+F 2 "TerminalBlock:TerminalBlock_bornier-4_P5.08mm" H 3950 4550 50  0001 C CNN
 F 3 "~" H 3950 4550 50  0001 C CNN
+F 4 "https://www.mouser.co.uk/ProductDetail/CUI-Devices/TB006-508-04BE?qs=vLWxofP3U2zpUvBkDCHiCA%3D%3D" H 3950 4550 50  0001 C CNN "Product"
 	1    3950 4550
 	-1   0    0    1
@@
 Wire Wire Line
 	4150 4650 4250 4650
+Wire Wire Line
+	1450 1900 1750 1900
+Wire Wire Line
+	1750 2100 1450 2100
+Wire Wire Line
+	1450 2200 1750 2200
+Wire Wire Line
+	1150 2550 1150 2700
 $EndSCHEMATC

Commit message: PCB Layout work
Parts:
- added J6: Screw_Terminal_01x06, TerminalBlock_Phoenix:TerminalBlock_Phoenix_MPT-0,5-6-2.54_1x06_P2.54mm_Horizontal, symbol Connector:Screw_Terminal_01x06
- J5: footprint TerminalBlock:TerminalBlock_bornier-4_P5.08mm -> TerminalBlock_Phoenix:TerminalBlock_Phoenix_MPT-0,5-4-2.54_1x04_P2.54mm_Horizontal
Connections:
- net +3.3V: now also J5.1 (Pin_1); no longer J5.2 (Pin_2)
- net AUDIO_L: now also J6.2 (Pin_2), J6.5 (Pin_5)
- net AUDIO_R: now also J6.1 (Pin_1), J6.6 (Pin_6)
- net Earth: now also J5.2 (Pin_2), J6.3 (Pin_3), J6.4 (Pin_4); no longer J5.4 (Pin_4)
- net LED_OUT: now also J5.4 (Pin_4); no longer J5.1 (Pin_1)
Changed lines of the file:
@@
 Text Label 6100 2400 2    50   ~ 0
 MSGEQ7_STROBE
-Text Label 4250 4650 0    50   ~ 0
+Text Label 4250 4350 0    50   ~ 0
 LED_OUT
 Text Label 4700 3050 0    50   ~ 0
@@
 Wire Wire Line
 	4500 1550 4700 1550
-$Comp
-L power:Earth #PWR05
-U 1 1 5F55AF8B
-P 4650 4350
-AR Path="/5F55AF8B" Ref="#PWR05"  Part="1"
-AR Path="/5F591C5D/5F55AF8B" Ref="#PWR?"  Part="1"
-F 0 "#PWR05" H 4650 4100 50  0001 C CNN
-F 1 "Earth" H 4650 4200 50  0001 C CNN
-F 2 "" H 4650 4350 50  0001 C CNN
-F 3 "~" H 4650 4350 50  0001 C CNN
-	1    4650 4350
-	0    -1   -1   0
-$EndComp
-Text Label 4250 4550 0    50   ~ 0
-+3.3V
 Text Label 4700 2950 0    50   ~ 0
 IR_SENSOR
 Wire Wire Line
 	4500 2950 4700 2950
-Text Label 4250 4450 0    50   ~ 0
-IR_SENSOR
 $Comp
 L SamacSys:SJ1-3523N J3
@@
 F 0 "J5" H 3868 4125 50  0000 C CNN
 F 1 "Screw_Terminal_01x04" H 3868 4216 50  0000 C CNN
-F 2 "TerminalBlock:TerminalBlock_bornier-4_P5.08mm" H 3950 4550 50  0001 C CNN
+F 2 "TerminalBlock_Phoenix:TerminalBlock_Phoenix_MPT-0,5-4-2.54_1x04_P2.54mm_Horizontal" H 3950 4550 50  0001 C CNN
 F 3 "~" H 3950 4550 50  0001 C CNN
 F 4 "https://www.mouser.co.uk/ProductDetail/CUI-Devices/TB006-508-04BE?qs=vLWxofP3U2zpUvBkDCHiCA%3D%3D" H 3950 4550 50  0001 C CNN "Product"
@@
 $EndComp
 Wire Wire Line
-	4150 4350 4650 4350
-Wire Wire Line
 	4150 4450 4250 4450
 Wire Wire Line
-	4150 4550 4250 4550
-Wire Wire Line
 	4150 4650 4250 4650
 Wire Wire Line
+	4150 4350 4250 4350
+Wire Wire Line
 	1450 1900 1750 1900
 Wire Wire Line
@@
 Wire Wire Line
 	1150 2550 1150 2700
+$Comp
+L Connector:Screw_Terminal_01x06 J6
+U 1 1 5F57EA02
+P 3950 5350
+F 0 "J6" H 3868 4825 50  0000 C CNN
+F 1 "Screw_Terminal_01x06" H 3868 4916 50  0000 C CNN
+F 2 "TerminalBlock_Phoenix:TerminalBlock_Phoenix_MPT-0,5-6-2.54_1x06_P2.54mm_Horizontal" H 3950 5350 50  0001 C CNN
+F 3 "~" H 3950 5350 50  0001 C CNN
+	1    3950 5350
+	-1   0    0    1
+$EndComp
+Wire Wire Line
+	4150 5250 4250 5250
+Wire Wire Line
+	4250 5250 4250 5350
+Wire Wire Line
+	4250 5350 4150 5350
+$Comp
+L power:Earth #PWR0101
+U 1 1 5F590EF5
+P 4250 5650
+AR Path="/5F590EF5" Ref="#PWR0101"  Part="1"
+AR Path="/5F591C5D/5F590EF5" Ref="#PWR?"  Part="1"
+F 0 "#PWR0101" H 4250 5400 50  0001 C CNN
+F 1 "Earth" H 4250 5500 50  0001 C CNN
+F 2 "" H 4250 5650 50  0001 C CNN
+F 3 "~" H 4250 5650 50  0001 C CNN
+	1    4250 5650
+	1    0    0    -1
+$EndComp
+Connection ~ 4250 5350
+Text Label 4450 5150 0    50   ~ 0
+AUDIO_L
+Wire Wire Line
+	4250 5350 4250 5650
+Wire Wire Line
+	4150 5150 4300 5150
+Wire Wire Line
+	4150 5450 4300 5450
+Wire Wire Line
+	4300 5450 4300 5150
+Wire Wire Line
+	4150 5050 4350 5050
+Wire Wire Line
+	4350 5050 4350 5550
+Wire Wire Line
+	4350 5550 4150 5550
+Text Label 4450 5050 0    50   ~ 0
+AUDIO_R
+Wire Wire Line
+	4450 5050 4350 5050
+Connection ~ 4350 5050
+Wire Wire Line
+	4450 5150 4300 5150
+Connection ~ 4300 5150
+Text Label 4250 4450 0    50   ~ 0
+IR_SENSOR
+$Comp
+L power:Earth #PWR05
+U 1 1 5F55AF8B
+P 4650 4550
+AR Path="/5F55AF8B" Ref="#PWR05"  Part="1"
+AR Path="/5F591C5D/5F55AF8B" Ref="#PWR?"  Part="1"
+F 0 "#PWR05" H 4650 4300 50  0001 C CNN
+F 1 "Earth" H 4650 4400 50  0001 C CNN
+F 2 "" H 4650 4550 50  0001 C CNN
+F 3 "~" H 4650 4550 50  0001 C CNN
+	1    4650 4550
+	0    -1   -1   0
+$EndComp
+Text Label 4250 4650 0    50   ~ 0
++3.3V
+Wire Wire Line
+	4150 4550 4650 4550
 $EndSCHEMATC
