File: PCB/Main_Board/Main_Board.kicad_pcb (KiCad board)
At the start: 2 copper layers, 68.2 x 58.2 mm, 62 parts, among them IC1 74LV1T34GVH, J1 USB_B_Micro, J2 Screw_Terminal_01x02, J3 SJ1-3523N, J4 SJ1-3523N, J5 Screw_Terminal_01x04, J6 Screw_Terminal_01x06, Q1 MBT3904DW1, SW1 SW_SPDT, SW2 EN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

Commit message: Update KiCAD to 5.1.7 and change a couple of footprints
Parts:
- added R11: 1k, Resistor_SMD:R_0603_1608Metric_Pad0.98x0.95mm_HandSolder, F.Cu at (120.7, 161.3)
- added R12: 1k, Resistor_SMD:R_0603_1608Metric_Pad0.98x0.95mm_HandSolder, F.Cu at (120.7, 163.8)
- C3: value 0.1uF -> 10uF
- J2: footprint TerminalBlock:TerminalBlock_bornier-2_P5.08mm -> Missing_Models:TerminalBlock_bornier-2_P5.08mm
- Q1: footprint Package_TO_SOT_SMD:SOT-363_SC-70-6 -> Package_TO_SOT_SMD:SOT-363_SC-70-6_Handsoldering
- R2: value 10k -> 47k
Connections:
- U4 pad 20: /ESP32_Circuit/IO3_RXD0 -> Net-(R11-Pad1)
- U4 pad 4: /ESP32_Circuit/IO1_TXD0 -> Net-(R12-Pad1)
Routing:
- net /ESP32_Circuit/EN: track 36.8 -> 37.5 mm
